Commit message: debug path in xacro

File: urdf/brov.xacro (robot description, xacro)
@@ -88,5 +88,5 @@
       <!--origin xyz="-0.241 0.165 0.17" rpy="${PI/2} 0 -${PI/2}"/-->
       <geometry>
-	<mesh filename="$(find bluerov_ffg)/mesh/brov-redux.stl" scale="0.001 0.001 0.001"/>
+	<mesh filename="file://$(find bluerov_ffg)/mesh/brov-redux.stl" scale="0.001 0.001 0.001"/>
       </geometry>
     </visual>

Commit message: with reduced mesh file

File: urdf/brov.xacro (robot description, xacro)
@@ -88,5 +88,5 @@
       <!--origin xyz="-0.241 0.165 0.17" rpy="${PI/2} 0 -${PI/2}"/-->
       <geometry>
-	<mesh filename="file://$(find bluerov_ffg)/mesh/brov-redux.stl" scale="0.001 0.001 0.001"/>
+	<mesh filename="file://$(find bluerov_ffg)/mesh/brov-redux.dae" scale="0.001 0.001 0.001"/>
       </geometry>
     </visual>

Commit message: with correct mesh file

File: urdf/brov.xacro (robot description, xacro)
@@ -88,5 +88,5 @@
       <!--origin xyz="-0.241 0.165 0.17" rpy="${PI/2} 0 -${PI/2}"/-->
       <geometry>
-	<mesh filename="file://$(find bluerov_ffg)/mesh/brov-redux.dae" scale="0.001 0.001 0.001"/>
+	<mesh filename="file://$(find bluerov_ffg)/mesh/brov-redux.stl" scale="0.001 0.001 0.001"/>
       </geometry>
     </visual>

Commit message: bad bad gains

File: urdf/brov.xacro (robot description, xacro)
@@ -102,10 +102,4 @@
 	  izz="5"/>
     </inertial>
-    <!--collision>
-      <origin xyz="0 0 0" rpy="0 0 0"/>
-      <geometry>
-	<box size="1 1 1"/>
-      </geometry>
-    </collision-->
   <buoyancy>
       <compensation>1.01</compensation>

Commit message: better thruster calibration

File: urdf/brov.xacro (robot description, xacro)
@@ -4,10 +4,12 @@
   <xacro:property name="PI" value="3.1415926535897931"/>
   <!-- Body properties -->
-  <xacro:property name="thr12_y" value="0.115"/>
-  <xacro:property name="thr34_x" value="0.18"/>
-  <xacro:property name="thr34_y" value="0.1092"/>
-  <xacro:property name="thr5_x" value="0.17"/>
-  <xacro:property name="thr6_x" value="0.039"/>
-  <xacro:property name="thr56_z" value="0.105"/>
+  <xacro:property name="thr12_y" value="0.109"/>
+  <xacro:property name="thr1234_z" value="-0.02"/>
+  <xacro:property name="thr34_x" value="0.165"/>
+  <xacro:property name="thr34_y" value="0.11"/>
+  <xacro:property name="thr5_x" value="-0.185"/>
+  <xacro:property name="thr5_z" value="-0.105"/>
+  <xacro:property name="thr6_x" value="0.028"/>
+  <xacro:property name="thr6_z" value="-0.127"/>
   <xacro:property name="eps" value="0.00000001"/>
   <!-- Thruster link -->
@@ -54,10 +56,10 @@
             <effort>40</effort>
             <name>thr1</name>
-            <map>1 0 0 0 0 ${-thr12_y}</map>
+            <map>1 0 0 0 0 ${thr12_y}</map>
         </thruster>
         <thruster>
             <effort>40</effort>
             <name>thr2</name>
-            <map>1 0 0 0 0 ${thr12_y}</map>
+            <map>1 0 0 0 0 ${-thr12_y}</map>
         </thruster>
         <thruster>
@@ -74,10 +76,10 @@
             <effort>30</effort>
             <name>thr5</name>
-            <map>0 0 -1 0 ${-thr5_x} 0</map>
+            <map>0 0 -1 0 ${thr5_x} 0</map>
         </thruster>
         <thruster>
             <effort>30</effort>
             <name>thr6</name>
-            <map>0 1 0 ${-thr56_z} 0 0</map>
+            <map>0 1 0 ${-thr6_z} 0 0</map>
         </thruster>
     </plugin>
@@ -85,5 +87,5 @@
   <link name="base_link">
     <visual>
-      <origin xyz="-0.241 0.165 0.17" rpy="${-PI/2} 0 -${PI/2}"/>
+      <origin xyz="-0.253 -0.167 -0.19" rpy="${PI/2} 0 ${PI/2}"/>
       <!--origin xyz="-0.241 0.165 0.17" rpy="${PI/2} 0 -${PI/2}"/-->
       <geometry>
@@ -92,5 +94,5 @@
     </visual>
      <inertial>
-      <origin xyz="0 0 0.1" rpy="0 0 0"/>
+      <origin xyz="0 0 -0.1" rpy="0 0 0"/>
       <mass value="5"/>
       <inertia
@@ -105,13 +107,13 @@
       <compensation>1.01</compensation>
       <origin xyz= "0 0 0"/>
-      <limit radius=".5"/>
+      <limit radius=".15"/>
       <damping xyz="50 100 60" rpy="50 50 50"/>
   </buoyancy>
   </link>
-<xacro:thruster_dummy_link name="thr1" xyz="0.0 0.115 0.0" rpy="-0.0 -1.57079632679 0.0"/>
-<xacro:thruster_dummy_link name="thr2" xyz="0.0 -0.115 0.0" rpy="-0.0 -1.57079632679 0.0"/>
-<xacro:thruster_dummy_link name="thr3" xyz="0.18 0.1092 0.0" rpy="0.0 -0.0 0.0"/>
-<xacro:thruster_dummy_link name="thr4" xyz="0.18 -0.1092 0.0" rpy="0.0 -0.0 0.0"/>
-<xacro:thruster_dummy_link name="thr5" xyz="-0.17 0.0 0.0" rpy="0.0 -0.0 0.0"/>
-<xacro:thruster_dummy_link name="thr6" xyz="0.0 0.0 0.105" rpy="1.57079632679 -0.0 0.0"/>
+<xacro:thruster_dummy_link name="thr1" xyz="0.0 ${-thr12_y} ${thr1234_z}" rpy="-0.0 -1.57079632679 0.0"/>
+<xacro:thruster_dummy_link name="thr2" xyz="0.0 ${thr12_y} ${thr1234_z}" rpy="-0.0 -1.57079632679 0.0"/>
+<xacro:thruster_dummy_link name="thr3" xyz="${thr34_x} ${-thr34_y} ${thr1234_z}" rpy="0.0 -0.0 0.0"/>
+<xacro:thruster_dummy_link name="thr4" xyz="${thr34_x} ${thr34_y} ${thr1234_z}" rpy="0.0 -0.0 0.0"/>
+<xacro:thruster_dummy_link name="thr5" xyz="${thr5_x} 0.0 ${thr5_z}" rpy="0.0 -0.0 0.0"/>
+<xacro:thruster_dummy_link name="thr6" xyz="${thr6_x} 0.0 ${thr6_z}" rpy="1.57079632679 -0.0 0.0"/>
 </robot>
