Commit message: modified origin of BlueROV2 visual frame

File: urdf/brov2.xacro (robot description, xacro)
@@ -1,17 +1,17 @@
 <?xml version="1.0"?>
-   <!-- STL-version of the URDF, used with gazebo for dynamic simulation  -->
+<!-- STL-version of the URDF, used with gazebo for dynamic simulation  -->
 <robot name="brov" xmlns:xacro="http://www.ros.org/wiki/xacro">
-  <xacro:property name="PI" value="3.1415926535897931"/>
-  <!-- Body properties -->
-  <xacro:property name="thr12_x" value="0.13"/>
-  <xacro:property name="thr12_y" value="0.10"/>
-  <xacro:property name="thr34_x" value="0.14"/>
-  <xacro:property name="thr34_y" value="0.11"/>
-  <xacro:property name="thr_z" value="-0.08"/>
-  <xacro:property name="thr12_theta" value="0.7"/>
-  <xacro:property name="thr34_theta" value="0.58"/>
-  <xacro:property name="thr56_y" value="0.11"/>
-  <xacro:property name="eps" value="0.00000001"/>
-  <!-- Thruster link -->
+<xacro:property name="PI" value="3.1415926535897931"/>
+<!-- Body properties -->
+<xacro:property name="thr12_x" value="0.125"/>
+<xacro:property name="thr12_y" value="0.115"/>
+<xacro:property name="thr34_x" value="0.15"/>
+<xacro:property name="thr34_y" value="0.11"/>
+<xacro:property name="thr_z" value="-0.07"/>
+<xacro:property name="thr12_theta" value="0.7"/>
+<xacro:property name="thr34_theta" value="0.6"/>
+<xacro:property name="thr56_y" value="0.11"/>
+<xacro:property name="eps" value="0.00000001"/>
+<!-- Thruster link -->
     <xacro:macro name="thruster_link" params="name xyz rpy">
         <joint name="${name}" type="fixed">
@@ -45,5 +45,5 @@
             </gazebo>
         </xacro:macro>
-  <!-- Plugin list -->
+<!-- Plugin list -->
     <gazebo>
     <!-- Gazebo plugin listens to the body-->
@@ -53,4 +53,5 @@
         <link>base_link</link>
         <!-- for each thruster, give the map to XYZ+RPY and the maximum effort -->
+        <!-- alternatively, give a link name + the maximum effort -->
         <thruster>
             <effort>40</effort>
@@ -79,30 +80,34 @@
     </plugin>
     </gazebo>
-  <link name="base_link">
+<link name="base_link">
+<!-- Origin of base_link is at the center of the cylinder  -->
     <visual>
-      <origin xyz="-0.24 -0.17 -0.19" rpy="${PI/2} 0 ${PI/2}"/>
-      <!--origin xyz="-0.241 0.165 0.17" rpy="${PI/2} 0 -${PI/2}"/-->
-      <geometry>
-	<mesh filename="file://$(find bluerov_ffg)/mesh/BROV2-rdx.stl" scale="0.001 0.001 0.001"/>
-      </geometry>
+    <geometry>
+    <mesh filename="file://$(find bluerov_ffg)/mesh/BROV2-rdx.stl"/>
+    </geometry>
     </visual>
-     <inertial>
-      <origin xyz="0 0 -0.1" rpy="0 0 0"/>
-      <mass value="5"/>
-      <inertia
-	  ixx="5"
-	  ixy="0.0"
-	  ixz="0.0"
-	  iyy="5"
-	  iyz="5"
-	  izz="5"/>
+    <inertial>
+    <origin xyz="0 0 -0.1" rpy="0 0 0"/>
+    <mass value="7.5"/>
+    <inertia
+    ixx="0.099"
+    ixy="0.0"
+    ixz="0.0056"
+    iyy="0.129"
+    iyz="0"
+    izz="0.16"/>
     </inertial>
-  <buoyancy>
-      <compensation>1.01</compensation>
-      <origin xyz= "0 0 0"/>
-      <limit radius=".15"/>
-      <damping xyz="50 100 60" rpy="50 50 50"/>
-  </buoyancy>
-  </link>
+    <fluid>
+    <density>1</density>
+    <origin xyz= "0 0 -0.04"/>
+    <buoyancy>
+    <compensation>1.01</compensation>
+    <limit radius=".15"/>
+    </buoyancy>
+<hydrodynamics>
+    <damping xyz="50 100 60" rpy="50 50 50"/>
+</hydrodynamics>
+    </fluid>
+</link>
 <xacro:thruster_link name="thr1" xyz="${thr12_x} ${-thr12_y} ${thr_z}" rpy="0.0 ${PI/2} ${thr12_theta}"/>
 <xacro:thruster_link name="thr2" xyz="${thr12_x} ${thr12_y} ${thr_z}" rpy="0.0 ${PI/2} ${-thr12_theta}"/>

Commit message: macro version of BlueROV 2 for integration in custom robots

File: urdf/brov2.xacro (robot description, xacro)
@@ -2,117 +2,7 @@
 <!-- STL-version of the URDF, used with gazebo for dynamic simulation  -->
 <robot name="brov" xmlns:xacro="http://www.ros.org/wiki/xacro">
-<xacro:property name="PI" value="3.1415926535897931"/>
-<!-- Body properties -->
-<xacro:property name="thr12_x" value="0.125"/>
-<xacro:property name="thr12_y" value="0.115"/>
-<xacro:property name="thr34_x" value="0.15"/>
-<xacro:property name="thr34_y" value="0.11"/>
-<xacro:property name="thr_z" value="-0.07"/>
-<xacro:property name="thr12_theta" value="0.7"/>
-<xacro:property name="thr34_theta" value="0.6"/>
-<xacro:property name="thr56_y" value="0.11"/>
-<xacro:property name="eps" value="0.00000001"/>
-<!-- Thruster link -->
-    <xacro:macro name="thruster_link" params="name xyz rpy">
-        <joint name="${name}" type="fixed">
-            <parent link="base_link"/>
-            <child link="${name}"/>
-            <origin rpy="${rpy}" xyz="${xyz}"/>
-        </joint>
-        <link name="${name}">
-            <buoyancy><compensation>1.0</compensation></buoyancy>
-            <!--visual name="${name}">
-                <geometry>
-                    <cylinder length=".5" radius=".01"/>
-                </geometry>
-                <material name="black">
-                    <color rgba="0 0 0 1"/>
-                </material>
-            </visual>
-            <inertial>
-                <mass value=".1"/>
-                <inertia
-                    ixx=".1"
-                    ixy="0.0"
-                    ixz="0.0"
-                    iyy=".1"
-                    iyz="0.0"
-                    izz=".1"/>
-                </inertial-->
-            </link>
-            <gazebo reference="${name}">
-                <material>Gazebo/Black</material>
-            </gazebo>
-        </xacro:macro>
-<!-- Plugin list -->
-    <gazebo>
-    <!-- Gazebo plugin listens to the body-->
-    <plugin name="freefloating_gazebo_control" filename="libfreefloating_gazebo_control.so">
-        <switchService>switch</switchService>
-        <updateRate>100</updateRate>
-        <link>base_link</link>
-        <!-- for each thruster, give the map to XYZ+RPY and the maximum effort -->
-        <!-- alternatively, give a link name + the maximum effort -->
-        <thruster>
-            <effort>40</effort>
-            <name>thr1</name>
-        </thruster>
-        <thruster>
-            <effort>40</effort>
-            <name>thr2</name>
-        </thruster>
-        <thruster>
-            <effort>30</effort>
-            <name>thr3</name>
-        </thruster>
-        <thruster>
-            <effort>30</effort>
-            <name>thr4</name>
-        </thruster>
-        <thruster>
-            <effort>30</effort>
-            <name>thr5</name>
-        </thruster>
-        <thruster>
-            <effort>30</effort>
-            <name>thr6</name>
-        </thruster>
-    </plugin>
-    </gazebo>
-<link name="base_link">
-<!-- Origin of base_link is at the center of the cylinder  -->
-    <visual>
-    <geometry>
-    <mesh filename="file://$(find bluerov_ffg)/mesh/BROV2-rdx.stl"/>
-    </geometry>
-    </visual>
-    <inertial>
-    <origin xyz="0 0 -0.1" rpy="0 0 0"/>
-    <mass value="7.5"/>
-    <inertia
-    ixx="0.099"
-    ixy="0.0"
-    ixz="0.0056"
-    iyy="0.129"
-    iyz="0"
-    izz="0.16"/>
-    </inertial>
-    <fluid>
-    <density>1</density>
-    <origin xyz= "0 0 -0.04"/>
-    <buoyancy>
-    <compensation>1.01</compensation>
-    <limit radius=".15"/>
-    </buoyancy>
-<hydrodynamics>
-    <damping xyz="50 100 60" rpy="50 50 50"/>
-</hydrodynamics>
-    </fluid>
-</link>
-<xacro:thruster_link name="thr1" xyz="${thr12_x} ${-thr12_y} ${thr_z}" rpy="0.0 ${PI/2} ${thr12_theta}"/>
-<xacro:thruster_link name="thr2" xyz="${thr12_x} ${thr12_y} ${thr_z}" rpy="0.0 ${PI/2} ${-thr12_theta}"/>
-<xacro:thruster_link name="thr3" xyz="${-thr34_x} ${-thr34_y} ${thr_z}" rpy="0.0 ${PI/2} ${PI-thr34_theta}"/>
-<xacro:thruster_link name="thr4" xyz="${-thr34_x} ${thr34_y} ${thr_z}" rpy="0.0 ${PI/2} ${PI+thr34_theta}"/>
-<xacro:thruster_link name="thr5" xyz="0.0 ${-thr56_y} 0" rpy="0.0 0 0.0"/>
-<xacro:thruster_link name="thr6" xyz="0.0 ${thr56_y} 0" rpy="0.0 0 0.0"/>
+<xacro:arg name="use_mesh" default="true"/>
+<xacro:arg name="density" default="1"/>
+<xacro:include filename="$(find bluerov_ffg)/urdf/brov2_macro.xacro"/>
+<xacro:generate_bluerov use_mesh="$(arg use_mesh)" density="$(arg density)" x_offset="0.02"/>
 </robot>
